File: plan/kicad/montageFinal/pvb/pvb.kicad_sch (KiCad schematic)
At the start: 0 parts

Commit message: modification du rapport final et des programme
Parts:
- added C?: C, symbol Device:C
- added R?: R, symbol Device:R
Changed lines of the file:
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@@
 (kicad_sch (version 20211123) (generator eeschema)
   (paper "A4")
+  (symbol (lib_id "Device:R") (at 91.44 68.58 0) (unit 1)
+    (in_bom yes) (on_board yes) (fields_autoplaced)
+    (property "Reference" "R?" (id 0) (at 93.98 67.3099 0)
+      (effects (font (size 1.27 1.27)) (justify left))
+    )
+    (property "Value" "R" (id 1) (at 93.98 69.8499 0)
+      (effects (font (size 1.27 1.27)) (justify left))
+    )
+    (property "Footprint" "" (id 2) (at 89.662 68.58 90)
+      (effects (font (size 1.27 1.27)) hide)
+    )
+    (property "Datasheet" "~" (id 3) (at 91.44 68.58 0)
+      (effects (font (size 1.27 1.27)) hide)
+    )
+    (pin "1")
+    (pin "2")
+  )
+  (symbol (lib_id "Device:C") (at 125.73 67.31 0) (unit 1)
+    (in_bom yes) (on_board yes) (fields_autoplaced)
+    (property "Reference" "C?" (id 0) (at 129.54 66.0399 0)
+      (effects (font (size 1.27 1.27)) (justify left))
+    )
+    (property "Value" "C" (id 1) (at 129.54 68.5799 0)
+      (effects (font (size 1.27 1.27)) (justify left))
+    )
+    (property "Footprint" "" (id 2) (at 126.6952 71.12 0)
+      (effects (font (size 1.27 1.27)) hide)
+    )
+    (property "Datasheet" "~" (id 3) (at 125.73 67.31 0)
+      (effects (font (size 1.27 1.27)) hide)
+    )
+    (pin "1")
+    (pin "2")
+  )
   (sheet_instances
     (path "/" (page "1"))
   )
+  (symbol_instances
+    (path "/cbed2fe2-862b-4775-b091-7fb7fee09cfd"
+      (reference "C?") (unit 1) (value "C") (footprint "")
+    )
+    (path "/5726890a-f461-4663-8372-3ae20d59de08"
+      (reference "R?") (unit 1) (value "R") (footprint "")
+    )
+  )
 )
